File: ESP32_lamp/ESP32_lamp.sch (KiCad schematic (older format))
At the start: 20 parts, among them U1 ESP32-WROOM-32D

Commit message: update repositories
Parts:
- removed D? (x4): LED, symbol Device:LED
- removed Q? (x4): 2N7002E, Package_TO_SOT_SMD:SOT-23, symbol Transistor_FET:2N7002E
- removed R?: R, symbol Device:R
- added 6.8, R4, R5, R6, R7, R8, R9: R, symbol Device:R
- added CB1: CircuitBreaker_1P_US, Jumper:SolderJumper-2_P1.3mm_Open_TrianglePad1.0x1.5mm, symbol Device:CircuitBreaker_1P_US
- added CB2: CircuitBreaker_1P, Jumper:SolderJumper-2_P1.3mm_Open_TrianglePad1.0x1.5mm, symbol Device:CircuitBreaker_1P
- added J1: Conn_02x05_Odd_Even, Connector_PinHeader_1.27mm:PinHeader_2x05_P1.27mm_Vertical, symbol Connector_Generic:Conn_02x05_Odd_Even
- added Q1, Q10, Q2, Q3, Q4, Q5, Q6, Q7, Q8, Q9: BSS214NW, Package_TO_SOT_SMD:SOT-323_SC-70, symbol Transistor_FET:BSS214NW
- added R10, R11: 6.8, symbol Device:R
- added U10: TPS62142, Package_DFN_QFN:VQFN-16-1EP_3x3mm_P0.5mm_EP1.68x1.68mm_ThermalVias, symbol Regulator_Switching:TPS62142
- added U3: CP2102N-A01-GQFN28, Package_DFN_QFN:QFN-28-1EP_5x5mm_P0.5mm_EP3.35x3.35mm, symbol Interface_USB:CP2102N-A01-GQFN28
- added U4: CP2102N-A01-GQFN24, Package_DFN_QFN:QFN-24-1EP_4x4mm_P0.5mm_EP2.6x2.6mm, symbol Interface_USB:CP2102N-A01-GQFN24
- added U5, U6, U7: AAAF5051-05, ESP32_lamp:kinbright-AAAF5051-05, symbol ESP_lamp:AAAF5051-05
- added U9: LM2576S-3.3, Package_TO_SOT_SMD:TO-263-5_TabPin3, symbol Regulator_Switching:LM2576S-3.3
- gave numbers to parts that had none: 7
Connections:
- net labels added: MTCK, MTDI, MTDO, MTMS
- wire segments 49 -> 111
- no-connect marks 0 -> 7
Other:
- moved on the sheet: C1, C100, C2, C3, D5, L1, R1, R2, R3, U1, U2

Commit message: update schem
Parts:
- removed 6.8, R1, R2, R3, R4, R5, R6, R7, R8, R9: R, symbol Device:R
- removed C1: 220u, symbol Device:CP_Small
- removed C100: 10u, symbol Device:C_Small
- removed C2: 0.1u, symbol Device:C_Small
- removed C3: 120u, symbol Device:CP_Small
- removed CB1: CircuitBreaker_1P_US, Jumper:SolderJumper-2_P1.3mm_Open_TrianglePad1.0x1.5mm, symbol Device:CircuitBreaker_1P_US
- removed CB2: CircuitBreaker_1P, Jumper:SolderJumper-2_P1.3mm_Open_TrianglePad1.0x1.5mm, symbol Device:CircuitBreaker_1P
- removed D5: 1N5822, Diode_THT:D_DO-201AD_P15.24mm_Horizontal, symbol Diode:1N5822
- removed J1: Conn_02x05_Odd_Even, Connector_PinHeader_1.27mm:PinHeader_2x05_P1.27mm_Vertical, symbol Connector_Generic:Conn_02x05_Odd_Even
- removed L1: 68u, symbol Device:L_Small
- removed Q1, Q10, Q2, Q3, Q4, Q5, Q6, Q7, Q8, Q9: BSS214NW, Package_TO_SOT_SMD:SOT-323_SC-70, symbol Transistor_FET:BSS214NW
- removed R10, R11: 6.8, symbol Device:R
- removed U1: ESP32-WROOM-32D, RF_Module:ESP32-WROOM-32, symbol RF_Module:ESP32-WROOM-32D
- removed U10: TPS62142, Package_DFN_QFN:VQFN-16-1EP_3x3mm_P0.5mm_EP1.68x1.68mm_ThermalVias, symbol Regulator_Switching:TPS62142
- removed U2: LM2595S-3.3, Package_TO_SOT_SMD:TO-263-5_TabPin3, symbol Regulator_Switching:LM2595S-3.3
- removed U3: CP2102N-A01-GQFN28, Package_DFN_QFN:QFN-28-1EP_5x5mm_P0.5mm_EP3.35x3.35mm, symbol Interface_USB:CP2102N-A01-GQFN28
- removed U4: CP2102N-A01-GQFN24, Package_DFN_QFN:QFN-24-1EP_4x4mm_P0.5mm_EP2.6x2.6mm, symbol Interface_USB:CP2102N-A01-GQFN24
- removed U5, U6, U7: AAAF5051-05, ESP32_lamp:kinbright-AAAF5051-05, symbol ESP_lamp:AAAF5051-05
- removed U9: LM2576S-3.3, Package_TO_SOT_SMD:TO-263-5_TabPin3, symbol Regulator_Switching:LM2576S-3.3
Connections:
- no-connect marks 7 -> 0

Commit message: Release Candidate 0
Parts:
- added H1, H2, H3, H4: MountingHole, MountingHole:MountingHole_3.2mm_M3_ISO7380, symbol Mechanical:MountingHole
Changed lines of the file:
@@
 F1 "peripherals.sch" 50
 $EndSheet
+$Comp
+L Graphic:Logo_Open_Hardware_Small #LOGO1
+U 1 1 5F3E331F
+P 1450 7250
+F 0 "#LOGO1" H 1450 7525 50  0001 C CNN
+F 1 "Logo_Open_Hardware_Small" H 1450 7025 50  0001 C CNN
+F 2 "Symbol:OSHW-Logo2_9.8x8mm_Copper" H 1450 7544 50  0000 C CNN
+F 3 "~" H 1450 7250 50  0001 C CNN
+	1    1450 7250
+	1    0    0    -1
+$EndComp
+$Comp
+L Mechanical:MountingHole H2
+U 1 1 5F3E89CB
+P 2450 7350
+F 0 "H2" H 2550 7396 50  0000 L CNN
+F 1 "MountingHole" H 2550 7305 50  0000 L CNN
+F 2 "MountingHole:MountingHole_3.2mm_M3_ISO7380" H 2450 7350 50  0001 C CNN
+F 3 "~" H 2450 7350 50  0001 C CNN
+	1    2450 7350
+	1    0    0    -1
+$EndComp
+$Comp
+L Mechanical:MountingHole H4
+U 1 1 5F3E8C67
+P 3000 7350
+F 0 "H4" H 3100 7396 50  0000 L CNN
+F 1 "MountingHole" H 3100 7305 50  0000 L CNN
+F 2 "MountingHole:MountingHole_3.2mm_M3_ISO7380" H 3000 7350 50  0001 C CNN
+F 3 "~" H 3000 7350 50  0001 C CNN
+	1    3000 7350
+	1    0    0    -1
+$EndComp
+$Comp
+L Mechanical:MountingHole H1
+U 1 1 5F3E8E0F
+P 2450 7100
+F 0 "H1" H 2550 7146 50  0000 L CNN
+F 1 "MountingHole" H 2550 7055 50  0000 L CNN
+F 2 "MountingHole:MountingHole_3.2mm_M3_ISO7380" H 2450 7100 50  0001 C CNN
+F 3 "~" H 2450 7100 50  0001 C CNN
+	1    2450 7100
+	1    0    0    -1
+$EndComp
+$Comp
+L Mechanical:MountingHole H3
+U 1 1 5F3E91C3
+P 3000 7100
+F 0 "H3" H 3100 7146 50  0000 L CNN
+F 1 "MountingHole" H 3100 7055 50  0000 L CNN
+F 2 "MountingHole:MountingHole_3.2mm_M3_ISO7380" H 3000 7100 50  0001 C CNN
+F 3 "~" H 3000 7100 50  0001 C CNN
+	1    3000 7100
+	1    0    0    -1
+$EndComp
 $EndSCHEMATC
