File: ESP32_lamp/Fuente_alimentacion.sch (KiCad schematic (older format))
At the start: 13 parts, among them J1 USB_B_Micro, U1 LMR33630BDDA

Commit message: Release Candidate 0
Parts:
- J1: MPN (none) -> 47590-0001
Changed lines of the file:
@@
 F 1 "USB_B_Micro" H 2607 3976 50  0000 C CNN
 F 2 "Connector_USB:USB_Micro-AB_Molex_47590-0001" H 2700 3550 50  0001 C CNN
-F 3 "~" H 2700 3550 50  0001 C CNN
+F 3 "https://www.mouser.es/datasheet/2/276/0475900001_IO_CONNECTORS-704847.pdf" H 2700 3550 50  0001 C CNN
+F 4 "47590-0001 " H 2550 3600 50  0001 C CNN "MPN"
 	1    2550 3600
 	1    0    0    -1
