File: ESP32_lamp/ESP32_&_LEDS.sch (KiCad schematic (older format))
At the start: 11 parts, among them J2 Conn_02x05_Odd_Even, J3 Conn_01x02, J4 Conn_01x03, U2 ESP32-WROOM-32D

Commit message: update
Parts:
- removed J3: Conn_01x02, symbol Connector_Generic:Conn_01x02
- added R6: 10k, Resistor_SMD:R_1206_3216Metric, symbol Device:R
- C11: value 0.1u -> 100nF
- J4: footprint (none) -> Connector_PinHeader_2.54mm:PinHeader_1x03_P2.54mm_Vertical_SMD_Pin1Left
Connections:
- net GND: now also R6.2; no longer CB1.2
- net SCL: now also U2.31 (IO19)
- net SDA: now also U2.33 (IO21)
- net LED_G3: now reaches U2.10 (IO25)
- net LED_B2: now reaches U2.11 (IO26)
- net LED_R2: now reaches U2.12 (IO27)
- net LED_G2: now reaches U2.26 (IO4)
- net LED_B1: now reaches U2.27 (IO16)
- net LED_R1: now reaches U2.28 (IO17)
- net LED_G1: now reaches U2.30 (IO18)
- net INT2: now reaches U2.36 (IO22)
- net INT1: now reaches U2.37 (IO23)
- net LED_B3: now reaches U2.8 (IO32)
- net LED_R3: now reaches U2.9 (IO33)
- new net: CB1.2, R6.1
Changed lines of the file:
@@
 Comment4 ""
 $EndDescr
-Wire Wire Line
-	3250 2900 3500 2900
 $Comp
 L power:GND #PWR?
 U 1 1 5F189CFB
-P 3700 2900
+P 4050 2900
 AR Path="/5F189CFB" Ref="#PWR?"  Part="1"
 AR Path="/5F10C517/5F189CFB" Ref="#PWR013"  Part="1"
-F 0 "#PWR013" H 3700 2650 50  0001 C CNN
-F 1 "GND" V 3705 2772 50  0000 R CNN
-F 2 "" H 3700 2900 50  0001 C CNN
-F 3 "" H 3700 2900 50  0001 C CNN
-	1    3700 2900
+F 0 "#PWR013" H 4050 2650 50  0001 C CNN
+F 1 "GND" V 4055 2772 50  0000 R CNN
+F 2 "" H 4050 2900 50  0001 C CNN
+F 3 "" H 4050 2900 50  0001 C CNN
+	1    4050 2900
 	0    -1   -1   0
 $EndComp
-Wire Wire Line
-	2650 2900 2600 2900
 $Comp
 L Device:CircuitBreaker_1P_US CB?
@@
 AR Path="/5F10C517/5F189D96" Ref="C11"  Part="1"
 F 0 "C11" V 1750 2450 50  0000 C CNN
-F 1 "0.1u" V 1750 2650 50  0000 C CNN
+F 1 "100nF" V 1750 2650 50  0000 C CNN
 F 2 "Capacitor_SMD:C_1206_3216Metric" H 1650 2550 50  0001 C CNN
 F 3 "~" H 1650 2550 50  0001 C CNN
@@
 F 0 "J4" H 4030 3192 50  0000 L CNN
 F 1 "Conn_01x03" H 4030 3101 50  0000 L CNN
-F 2 "" H 3950 3150 50  0001 C CNN
+F 2 "Connector_PinHeader_2.54mm:PinHeader_1x03_P2.54mm_Vertical_SMD_Pin1Left" H 3950 3150 50  0001 C CNN
 F 3 "~" H 3950 3150 50  0001 C CNN
 	1    3950 3150
@@
 MTDI
 NoConn ~ 2150 6900
-$Comp
-L Connector_Generic:Conn_01x02 J3
-U 1 1 5F1D49BB
-P 3850 2350
-F 0 "J3" H 3930 2342 50  0000 L CNN
-F 1 "Conn_01x02" H 3930 2251 50  0000 L CNN
-F 2 "" H 3850 2350 50  0001 C CNN
-F 3 "~" H 3850 2350 50  0001 C CNN
-	1    3850 2350
-	1    0    0    -1
-$EndComp
 Wire Wire Line
 	1750 2250 1900 2250
@@
 Connection ~ 1450 2400
 Wire Wire Line
-	2600 2350 2600 2900
-Wire Wire Line
-	2600 2350 3650 2350
-Connection ~ 2600 2900
-Wire Wire Line
-	2600 2900 2500 2900
-Wire Wire Line
-	3650 2450 3500 2450
-Wire Wire Line
-	3500 2450 3500 2900
-Connection ~ 3500 2900
-Wire Wire Line
-	3500 2900 3700 2900
-Wire Wire Line
 	2500 3000 3600 3000
 Text GLabel 4700 6400 3    50   Input ~ 0
@@
 Text GLabel 1900 2100 1    50   Input ~ 0
 3V3
+Wire Wire Line
+	2500 5000 2750 5000
+Wire Wire Line
+	2500 4900 2750 4900
+Wire Wire Line
+	2500 4600 2750 4600
+Wire Wire Line
+	2500 4700 2750 4700
+Wire Wire Line
+	2500 4800 2750 4800
+Text GLabel 2750 4900 2    50   Output ~ 0
+LED_B3
+Text GLabel 2750 5000 2    50   Output ~ 0
+LED_R3
+Text GLabel 2750 4600 2    50   Output ~ 0
+LED_G3
+Text GLabel 2750 4700 2    50   Output ~ 0
+LED_B2
+Text GLabel 2750 4800 2    50   Output ~ 0
+LED_R2
+Wire Wire Line
+	2500 3300 2750 3300
+Text GLabel 2750 3300 2    50   Output ~ 0
+LED_G2
+Wire Wire Line
+	2500 3900 2750 3900
+Text GLabel 2750 3900 2    50   Output ~ 0
+LED_B1
+Wire Wire Line
+	2500 4000 2750 4000
+Text GLabel 2750 4000 2    50   Output ~ 0
+LED_R1
+Wire Wire Line
+	2500 4100 2750 4100
+Text GLabel 2750 4100 2    50   Output ~ 0
+LED_G1
+Text GLabel 2850 4300 2    50   Output ~ 0
+SDA
+Text GLabel 2850 4200 2    50   Output ~ 0
+SCL
+Wire Wire Line
+	2500 4200 2850 4200
+Wire Wire Line
+	2500 4300 2850 4300
+Wire Wire Line
+	2500 2900 2650 2900
+Wire Wire Line
+	3250 2900 3450 2900
+$Comp
+L Device:R R?
+U 1 1 5F24588B
+P 3600 2900
+AR Path="/5F24588B" Ref="R?"  Part="1"
+AR Path="/5F10C517/5F24588B" Ref="R6"  Part="1"
+F 0 "R6" V 3393 2900 50  0000 C CNN
+F 1 "10k" V 3484 2900 50  0000 C CNN
+F 2 "Resistor_SMD:R_1206_3216Metric" V 3530 2900 50  0001 C CNN
+F 3 "~" H 3600 2900 50  0001 C CNN
+	1    3600 2900
+	0    -1   -1   0
+$EndComp
+Wire Wire Line
+	3750 2900 4050 2900
+Wire Wire Line
+	2500 4400 2750 4400
+Wire Wire Line
+	2500 4500 2750 4500
+Text GLabel 2750 4400 2    50   Input ~ 0
+INT2
+Text GLabel 2750 4500 2    50   Input ~ 0
+INT1
 $EndSCHEMATC

Commit message: WIP Release Candidate 1
Parts:
- added C16: 100nF, Capacitor_SMD:C_1206_3216Metric, symbol Device:C_Small
- added R7: 10k, Resistor_SMD:R_1206_3216Metric, symbol Device:R
- added SW1: SW_Push, Button_Switch_SMD:Panasonic_EVQPUJ_EVQPUA, symbol Switch:SW_Push
Connections:
- wire segments 69 -> 78
Changed lines of the file:
@@
 	2500 4300 2850 4300
 Wire Wire Line
-	2500 2900 2650 2900
+	2500 2900 2550 2900
 Wire Wire Line
 	3250 2900 3450 2900
@@
 Text GLabel 2750 4500 2    50   Input ~ 0
 INT1
+$Comp
+L Device:R R?
+U 1 1 5F46936E
+P 5000 2100
+AR Path="/5F46936E" Ref="R?"  Part="1"
+AR Path="/5F10C517/5F46936E" Ref="R7"  Part="1"
+F 0 "R7" V 4793 2100 50  0000 C CNN
+F 1 "10k" V 4884 2100 50  0000 C CNN
+F 2 "Resistor_SMD:R_1206_3216Metric" V 4930 2100 50  0001 C CNN
+F 3 "~" H 5000 2100 50  0001 C CNN
+	1    5000 2100
+	1    0    0    -1
+$EndComp
+Wire Wire Line
+	5000 2250 5000 2400
+Wire Wire Line
+	5000 2400 2550 2400
+Wire Wire Line
+	2550 2400 2550 2900
+Connection ~ 5000 2400
+Connection ~ 2550 2900
+Wire Wire Line
+	2550 2900 2650 2900
+Text GLabel 5000 1850 1    50   Input ~ 0
+3V3
+Wire Wire Line
+	5000 1850 5000 1950
+$Comp
+L power:GND #PWR?
+U 1 1 5F470D31
+P 5550 2700
+AR Path="/5F470D31" Ref="#PWR?"  Part="1"
+AR Path="/5F10C517/5F470D31" Ref="#PWR0104"  Part="1"
+F 0 "#PWR0104" H 5550 2450 50  0001 C CNN
+F 1 "GND" V 5555 2572 50  0000 R CNN
+F 2 "" H 5550 2700 50  0001 C CNN
+F 3 "" H 5550 2700 50  0001 C CNN
+	1    5550 2700
+	1    0    0    -1
+$EndComp
+$Comp
+L Device:C_Small C?
+U 1 1 5F472DB2
+P 5000 2650
+AR Path="/5F472DB2" Ref="C?"  Part="1"
+AR Path="/5F10C517/5F472DB2" Ref="C16"  Part="1"
+F 0 "C16" V 5100 2550 50  0000 C CNN
+F 1 "100nF" V 5100 2750 50  0000 C CNN
+F 2 "Capacitor_SMD:C_1206_3216Metric" H 5000 2650 50  0001 C CNN
+F 3 "~" H 5000 2650 50  0001 C CNN
+	1    5000 2650
+	1    0    0    -1
+$EndComp
+$Comp
+L power:GND #PWR?
+U 1 1 5F4737E0
+P 5000 2900
+AR Path="/5F4737E0" Ref="#PWR?"  Part="1"
+AR Path="/5F10C517/5F4737E0" Ref="#PWR0105"  Part="1"
+F 0 "#PWR0105" H 5000 2650 50  0001 C CNN
+F 1 "GND" V 5005 2772 50  0000 R CNN
+F 2 "" H 5000 2900 50  0001 C CNN
+F 3 "" H 5000 2900 50  0001 C CNN
+	1    5000 2900
+	1    0    0    -1
+$EndComp
+Wire Wire Line
+	5000 2900 5000 2750
+Wire Wire Line
+	5000 2550 5000 2400
+$Comp
+L Switch:SW_Push SW1
+U 1 1 5F468DD6
+P 5350 2400
+F 0 "SW1" H 5350 2685 50  0000 C CNN
+F 1 "SW_Push" H 5350 2594 50  0000 C CNN
+F 2 "Button_Switch_SMD:Panasonic_EVQPUJ_EVQPUA" H 5350 2600 50  0001 C CNN
+F 3 "~" H 5350 2600 50  0001 C CNN
+	1    5350 2400
+	-1   0    0    -1
+$EndComp
+Wire Wire Line
+	5150 2400 5000 2400
+Wire Wire Line
+	5550 2700 5550 2400
 $EndSCHEMATC
