File: ESP32_lamp/ESP32_lamp.kicad_pcb (KiCad board)
At the start: 2 copper layers, 100 x 100 mm, 23 parts, among them J1 Conn_02x05_Odd_Even, Q1 BSS214NW, Q10 BSS214NW, Q2 BSS214NW, Q3 BSS214NW, Q4 BSS214NW, Q5 BSS214NW, Q6 BSS214NW, Q7 BSS214NW, Q8 BSS214NW, Q9 BSS214NW, U1 ESP32-WROOM-32D, U10 TPS62142, U2 LM2595S-3.3, U3 CP2102N-A01-GQFN28, U4 CP2102N-A01-GQFN24, U5 AAAF5051-05, U6 AAAF5051-05, U7 AAAF5051-05, U9 LM2576S-3.3

Commit message: update schem
Parts:
- removed CB2: CircuitBreaker_1P, Jumper:SolderJumper-2_P1.3mm_Open_TrianglePad1.0x1.5mm
- removed D5: 1N5822, Diode_THT:D_DO-201AD_P15.24mm_Horizontal
- removed Q1, Q10, Q2, Q3, Q4, Q5, Q6: BSS214NW, Package_TO_SOT_SMD:SOT-323_SC-70
- removed U10: TPS62142, Package_DFN_QFN:VQFN-16-1EP_3x3mm_P0.5mm_EP1.68x1.68mm_ThermalVias
- removed U7: AAAF5051-05, ESP32_lamp:kinbright-AAAF5051-05
- removed U9: LM2576S-3.3, Package_TO_SOT_SMD:TO-263-5_TabPin3
- added C1: 10uF, Capacitor_SMD:C_1206_3216Metric, B.Cu at (128.0, 131.0)
- added C10: 10uF, Capacitor_SMD:C_1206_3216Metric, B.Cu at (144.0, 136.0)
- added C11: 0.1u, Capacitor_SMD:C_1206_3216Metric, B.Cu at (141.5, 136.0)
- added C2: 220nF, Capacitor_SMD:C_1206_3216Metric, B.Cu at (130.6, 131.0)
- added C3: 1uF, Capacitor_SMD:C_1206_3216Metric, B.Cu at (128.0, 118.0)
- added C4: 100nF, Capacitor_SMD:C_1206_3216Metric, B.Cu at (131.5, 118.2)
- added C5: 22uF, Capacitor_SMD:C_1206_3216Metric, B.Cu at (136.5, 127.9)
- added C6: 22uF, Capacitor_SMD:C_1206_3216Metric, B.Cu at (139.0, 128.0)
- added C7: 22uF, Capacitor_SMD:C_1206_3216Metric, B.Cu at (134.0, 128.0)
- added C8: 22uF, Capacitor_SMD:C_1206_3216Metric, B.Cu at (141.5, 127.9)
- added C9: 0.1uF, Capacitor_SMD:C_1206_3216Metric, B.Cu at (146.5, 136.0)
- added J2: Conn_02x05_Odd_Even, Connector_PinHeader_1.27mm:PinHeader_2x05_P1.27mm_Vertical_SMD, B.Cu at (126.8, 96.0)
- added L1: 2.2uH, 11.4mΩ, Inductor_SMD:L_Taiyo-Yuden_MD-5050, B.Cu at (135.5, 122.4)
- added Q_B1: BSS214NW, Package_TO_SOT_SMD:SOT-323_SC-70, F.Cu at (162.0, 107.0)
- added Q_B2: BSS214NW, Package_TO_SOT_SMD:SOT-323_SC-70, F.Cu at (152.0, 103.5)
- added Q_G1: BSS214NW, Package_TO_SOT_SMD:SOT-323_SC-70, F.Cu at (162.0, 113.0)
- added Q_G2: BSS214NW, Package_TO_SOT_SMD:SOT-323_SC-70, F.Cu at (158.0, 103.5)
- added Q_R1: BSS214NW, Package_TO_SOT_SMD:SOT-323_SC-70, F.Cu at (162.0, 110.0)
- added Q_R2: BSS214NW, Package_TO_SOT_SMD:SOT-323_SC-70, F.Cu at (155.0, 103.5)
- added R1: 100kΩ, Resistor_SMD:R_1206_3216Metric, B.Cu at (125.5, 118.0)
- added R2: 43.3kΩ, Resistor_SMD:R_1206_3216Metric, B.Cu at (125.5, 123.0)
- added R3: 10k, Resistor_SMD:R_1206_3216Metric, B.Cu at (145.2, 132.2)
- added R4: 10k, Resistor_SMD:R_1206_3216Metric, B.Cu at (185.0, 126.5)
- added R5: 10k, Resistor_SMD:R_1206_3216Metric, F.Cu at (185.0, 123.0)
- added R_B11: 220R, Resistor_SMD:R_1206_3216Metric, F.Cu at (159.2, 127.5)
- added R_B12: 0R, Resistor_SMD:R_1206_3216Metric, F.Cu at (166.5, 107.5)
- added R_B21: 220R, Resistor_SMD:R_1206_3216Metric, F.Cu at (151.5, 127.5)
- added R_B22: 0R, Resistor_SMD:R_1206_3216Metric, F.Cu at (152.2, 98.8)
- added R_B31: 220R, Resistor_SMD:R_1206_3216Metric, F.Cu at (144.0, 127.6)
- added R_B32: 0R, Resistor_SMD:R_1206_3216Metric, F.Cu at (142.6, 112.5)
- added R_G11: 220R, Resistor_SMD:R_1206_3216Metric, F.Cu at (164.2, 127.5)
- added R_G12: 0R, Resistor_SMD:R_1206_3216Metric, F.Cu at (166.5, 112.5)
- added R_G21: 220R, Resistor_SMD:R_1206_3216Metric, F.Cu at (156.5, 127.5)
- added R_G22: 0R, Resistor_SMD:R_1206_3216Metric, F.Cu at (157.8, 98.8)
- added R_G31: 220R, Resistor_SMD:R_1206_3216Metric, F.Cu at (149.0, 127.5)
- added R_G32: 0R, Resistor_SMD:R_1206_3216Metric, F.Cu at (142.7, 107.5)
- added R_R11: 220R, Resistor_SMD:R_1206_3216Metric, F.Cu at (161.8, 127.5)
- added R_R12: 6.8R, Resistor_SMD:R_1206_3216Metric, F.Cu at (166.5, 110.0)
- added R_R21: 220R, Resistor_SMD:R_1206_3216Metric, F.Cu at (154.0, 127.5)
- added R_R22: 6.8R, Resistor_SMD:R_1206_3216Metric, F.Cu at (155.0, 98.8)
- added R_R31: 220R, Resistor_SMD:R_1206_3216Metric, F.Cu at (146.5, 127.5)
- added R_R32: 6.8R, Resistor_SMD:R_1206_3216Metric, F.Cu at (142.6, 110.0)
- J1: value Conn_02x05_Odd_Even -> USB_B_Micro; footprint Connector_PinHeader_1.27mm:PinHeader_2x05_P1.27mm_Vertical -> Connector_USB:USB_Micro-AB_Molex_47590-0001; moved to B.Cu
- U1: value ESP32-WROOM-32D -> LMR33630BDDA; footprint RF_Module:ESP32-WROOM-32 -> Package_SO:Texas_HSOP-8-1EP_3.9x4.9mm_P1.27mm_ThermalVias; moved to B.Cu
- U2: value LM2595S-3.3 -> ESP32-WROOM-32D; footprint Package_TO_SOT_SMD:TO-263-5_TabPin3 -> RF_Module:ESP32-WROOM-32; moved to B.Cu
- U3: value CP2102N-A01-GQFN28 -> ADXL343; footprint Package_DFN_QFN:QFN-28-1EP_5x5mm_P0.5mm_EP3.35x3.35mm -> Package_LGA:LGA-14_3x5mm_P0.8mm_LayoutBorder1x6y; moved to B.Cu
- U4: value CP2102N-A01-GQFN24 -> AAAF5051-05; footprint Package_DFN_QFN:QFN-24-1EP_4x4mm_P0.5mm_EP2.6x2.6mm -> ESP32_lamp:kinbright-AAAF5051-05
- U5, U6: moved to F.Cu
- moved U2 96.9 mm to (158.0, 129.0)
- moved Q9 93.1 mm to (147.0, 107.5), turned to 180 degrees
- moved Q7 92.5 mm to (147.0, 112.5), turned to 180 degrees
- moved Q8 84.6 mm to (147.0, 110.0), turned to 180 degrees
- moved U6 80.4 mm to (134.5, 110.0), turned to 0 degrees
- moved J1 51.4 mm to (121.5, 130.6), turned to 90 degrees
- moved U1 32.6 mm to (129.6, 124.7)
- moved U4 32.1 mm to (175.0, 110.0), turned to 180 degrees
- moved CB1 24.3 mm to (176.5, 128.0), turned to 90 degrees
- moved U3 15.7 mm to (184.5, 131.0), turned to 180 degrees
- moved U5 15.6 mm to (155.0, 90.5), turned to 270 degrees
Connections:
- net Net-(U3-Pad8) renamed INT1
- net Net-(U3-Pad9) renamed INT2
- J1 pad 1: +3V3 -> VIN
- J1 pad 2: MTMS -> Net-(J1-Pad2)
- J1 pad 3: GND -> Net-(J1-Pad3)
- J1 pad 4: MTCK -> Net-(J1-Pad4)
- J1 pad 6: MTDO -> GND
- U1 pad 2: +3V3 -> VIN
- U1 pad 3: Net-(U1-Pad3) -> VIN
- U1 pad 9: Net-(U1-Pad9) -> GND
- U2 pad 1: Net-(D5-Pad1) -> GND
- U2 pad 2: +12V -> 3V3
- U2 pad 3: GND -> Net-(C9-Pad2)
- U2 pad 4: +3V3 -> Net-(U2-Pad4)
- U2 pad 5: GND -> Net-(U2-Pad5)
- U3 pad 1: Net-(U3-Pad1) -> 3V3
- U3 pad 11: Net-(U3-Pad11) -> GND
- U3 pad 12: Net-(U3-Pad12) -> GND
- U3 pad 13: Net-(U3-Pad13) -> SDA
- U3 pad 14: Net-(U3-Pad14) -> SCL
- U3 pad 2: Net-(U3-Pad2) -> GND
- U3 pad 3: Net-(U3-Pad29) -> 3V3
- U3 pad 4: Net-(U3-Pad4) -> GND
- U3 pad 5: Net-(U3-Pad5) -> GND
- U3 pad 6: Net-(U3-Pad6) -> 3V3
- U3 pad 7: Net-(U3-Pad7) -> 3V3
- U4 pad 4: Net-(U4-Pad4) -> 3V3_SW
- U4 pad 5: Net-(U4-Pad5) -> 3V3_SW
- U4 pad 6: Net-(U4-Pad6) -> 3V3_SW
- U4 pad 7: Net-(U4-Pad7) -> 3V3_SW
- U5 pad 4: +3V3 -> 3V3_SW
- U5 pad 5: +3V3 -> 3V3_SW
- U5 pad 6: +3V3 -> 3V3_SW
- U5 pad 7: +3V3 -> 3V3_SW
- U6 pad 3: Net-(Q7-Pad3) -> Net-(R_G32-Pad2)
- U6 pad 4: +3V3 -> 3V3_SW
- U6 pad 5: +3V3 -> 3V3_SW
- U6 pad 6: +3V3 -> 3V3_SW
- U6 pad 7: +3V3 -> 3V3_SW
Routing:
- net 3V3_SW: track 0.00 -> 85.5 mm, vias 0 -> 1
- net 3V3: track 0.00 -> 61.3 mm
- net GND: track 0.00 -> 59.9 mm, vias 0 -> 9
- net +3V3: track 23.3 -> 0.00 mm
- net Net-(Q_B1-Pad1): track 0.00 -> 22.7 mm
- net Net-(Q_B2-Pad1): track 0.00 -> 22.3 mm
- net Net-(Q_G2-Pad1): track 0.00 -> 22.0 mm
- net Net-(Q_R2-Pad1): track 0.00 -> 21.7 mm
- net Net-(Q9-Pad1): track 0.00 -> 21.0 mm
- net Net-(Q_R1-Pad1): track 0.00 -> 19.2 mm
- net Net-(Q8-Pad1): track 0.00 -> 18.9 mm
- net Net-(Q_G1-Pad1): track 0.00 -> 16.6 mm
- net Net-(Q7-Pad1): track 0.00 -> 14.7 mm
- net VIN: track 0.00 -> 12.6 mm
- net Net-(C4-Pad1): track 0.00 -> 11.8 mm
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- added copper zone on F.Cu, net 3V3
- added copper zone on B.Cu, net GND
- removed copper zone on B.Cu, net +3V3
Other:
- board size 100 x 100 mm -> 70 x 70 mm
- net class mediomm added: clearance 0.2, trace_width 0.5, via_dia 0.8, via_drill 0.4

Commit message: update
Parts:
- added C12: 100nF, Capacitor_SMD:C_1206_3216Metric, B.Cu at (179.0, 130.6)
- added G***: LOGO, ESP32_lamp:logo, F.Cu at (154.8, 131.0)
- added J4: Conn_01x03, Connector_PinHeader_2.54mm:PinHeader_1x03_P2.54mm_Vertical_SMD_Pin1Left, B.Cu at (185.6, 127.6)
- added R6: 10k, Resistor_SMD:R_1206_3216Metric, B.Cu at (174.0, 120.8)
- C11: value 0.1u -> 100nF
- CB1, R5: moved to B.Cu
- moved J2 62.2 mm to (185.2, 117.2), turned to 180 degrees
- moved R4 15.2 mm to (169.8, 125.5), turned to 90 degrees
- moved R5 12.8 mm to (172.4, 125.5), turned to 90 degrees
- moved U3 9.90 mm to (174.6, 130.8), turned to 270 degrees
- moved CB1 9.70 mm to (170.0, 120.8), turned to 0 degrees
- moved C8 8.59 mm to (136.0, 134.5), turned to 180 degrees
- moved R_B11 6.75 mm to (159.2, 120.8)
- moved R_B21 6.75 mm to (151.5, 120.8)
- moved R_B31 6.75 mm to (144.0, 120.8)
- moved R_G11 6.75 mm to (164.2, 120.8)
- moved R_G21 6.75 mm to (156.5, 120.8)
- moved R_G31 6.75 mm to (149.0, 120.8)
- moved R_R11 6.75 mm to (161.8, 120.8)
- moved R_R21 6.75 mm to (154.0, 120.8)
- moved R_R31 6.75 mm to (146.5, 120.8)
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Connections:
- CB1 pad 2: GND -> Net-(CB1-Pad2)
- U2 pad 10: Net-(U2-Pad10) -> LED_G3
- U2 pad 11: Net-(U2-Pad11) -> LED_B2
- U2 pad 12: Net-(U2-Pad12) -> LED_R2
- U2 pad 26: Net-(U2-Pad26) -> LED_G2
- U2 pad 27: Net-(U2-Pad27) -> LED_B1
- U2 pad 28: Net-(U2-Pad28) -> LED_R1
- U2 pad 30: Net-(U2-Pad30) -> LED_G1
- U2 pad 31: Net-(U2-Pad31) -> SCL
- U2 pad 33: Net-(U2-Pad33) -> SDA
- U2 pad 8: Net-(U2-Pad8) -> LED_B3
- U2 pad 9: Net-(U2-Pad9) -> LED_R3
Routing:
- net 3V3: track 61.3 -> 105.9 mm, vias 0 -> 2
- net MTMS: track 0.00 -> 43.6 mm
- net MTDI: track 0.00 -> 39.4 mm, vias 0 -> 2
- net MTCK: track 0.00 -> 32.0 mm
- net Net-(J4-Pad2): track 0.00 -> 25.3 mm
- net MTDO: track 0.00 -> 22.7 mm
- net Net-(J4-Pad1): track 0.00 -> 20.0 mm
- net SCL: track 0.00 -> 15.0 mm
- net LED_G2: track 0.00 -> 12.7 mm, vias 0 -> 1
- net SDA: track 0.00 -> 12.2 mm
- net LED_B3: track 0.00 -> 10.1 mm, vias 0 -> 1
- net LED_B1: track 0.00 -> 9.40 mm, vias 0 -> 1
- net Net-(Q_G1-Pad1): track 16.6 -> 8.35 mm
- net LED_R3: track 0.00 -> 7.45 mm, vias 0 -> 1
- net LED_R1: track 0.00 -> 7.12 mm, vias 0 -> 1
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
Commit message: Release Candidate 0
Parts:
- removed G***: LOGO, ESP32_lamp:logo
- added C13: 1uF, Capacitor_SMD:C_1206_3216Metric, F.Cu at (155.2, 83.0)
- added C14: 1uF, Capacitor_SMD:C_1206_3216Metric, F.Cu at (127.2, 110.0)
- added C15: 1uF, Capacitor_SMD:C_1206_3216Metric, F.Cu at (182.8, 110.2)
- added H1: MountingHole, MountingHole:MountingHole_3.2mm_M3_ISO7380, F.Cu at (125.0, 140.0)
- added H2: MountingHole, MountingHole:MountingHole_3.2mm_M3_ISO7380, F.Cu at (185.0, 140.0)
- added H3: MountingHole, MountingHole:MountingHole_3.2mm_M3_ISO7380, F.Cu at (184.9, 80.1)
- added H4: MountingHole, MountingHole:MountingHole_3.2mm_M3_ISO7380, F.Cu at (125.0, 80.0)
- added REF**: OSHW-Logo2_9.8x8mm_SilkScreen, Symbol:OSHW-Logo2_9.8x8mm_SilkScreen, B.Cu at (182.8, 89.1)
- added REF**: OSHW-Logo2_9.8x8mm_SilkScreen, Symbol:OSHW-Logo2_9.8x8mm_SilkScreen, F.Cu at (126.7, 89.3)
- renumbered U4 to LED1, U5 to LED2, U6 to LED3, Q7 to Q_B3, Q9 to Q_G3, Q8 to Q_R3
Connections:
- LED1 pad 4: 3V3_SW -> 3V3
- LED1 pad 5: 3V3_SW -> 3V3
- LED1 pad 6: 3V3_SW -> 3V3
- LED1 pad 7: 3V3_SW -> 3V3
- LED2 pad 4: 3V3_SW -> 3V3
- LED2 pad 5: 3V3_SW -> 3V3
- LED2 pad 6: 3V3_SW -> 3V3
- LED2 pad 7: 3V3_SW -> 3V3
- LED3 pad 4: 3V3_SW -> 3V3
- LED3 pad 5: 3V3_SW -> 3V3
- LED3 pad 6: 3V3_SW -> 3V3
- LED3 pad 7: 3V3_SW -> 3V3
- U2 pad 36: Net-(U2-Pad36) -> INT2
- U2 pad 37: Net-(U2-Pad37) -> INT1
Routing:
- net 3V3: track 105.9 -> 219.1 mm, vias 2 -> 7
- net 3V3_SW: track 85.5 -> 0.00 mm, vias 1 -> 0
- net GND: track 62.2 -> 114.2 mm, vias 14 -> 33
- net INT1: track 0.00 -> 14.4 mm, vias 0 -> 2
- net INT2: track 0.00 -> 13.7 mm, vias 0 -> 2
- net Net-(J4-Pad1): track 20.0 -> 21.3 mm
- net Net-(J4-Pad2): track 25.3 -> 26.3 mm
Other:
- board text added: "OSHW License"
- board text added: "https://github.com/zerberros/esp32_LAMP"

Commit message: Added backSilkscreen
Parts:
- removed the REF** at (182.8, 89.1)
Other:
- board text added: "esp32_lamp v20.08"

Commit message: Release
Parts:
- removed REF**: OSHW-Logo2_9.8x8mm_SilkScreen, Symbol:OSHW-Logo2_9.8x8mm_SilkScreen
- added C16: 100nF, Capacitor_SMD:C_1206_3216Metric, B.Cu at (185.0, 121.0)
- added R7: 10k, Resistor_SMD:R_1206_3216Metric, B.Cu at (183.6, 116.6)
- added SW1: SW_Push, Button_Switch_SMD:Panasonic_EVQPUJ_EVQPUA, B.Cu at (187.9, 115.2)
- LED1, LED2, LED3: footprint ESP32_lamp:kinbright-AAAF5051-05 -> ESP32_lamp:kinbright-AAAF5051-05_MOD
- moved J2 30.5 mm to (155.0, 113.4), turned to 270 degrees
- moved Q_B3 0.30 mm to (147.0, 112.8)
- moved Q_G3 0.30 mm to (147.0, 107.2)
Routing:
- net 3V3: track 219.1 -> 113.8 mm, vias 7 -> 8
- net MTMS: track 43.6 -> 9.21 mm
- net Net-(C16-Pad1): track 2.80 -> 33.0 mm
- net MTCK: track 32.0 -> 3.57 mm
- net GND: track 114.2 -> 141.8 mm, vias 33 -> 42
- net MTDI: track 39.4 -> 14.4 mm, vias 2 -> 0
- net MTDO: track 22.7 -> 10.9 mm
- net Net-(J4-Pad1): track 21.3 -> 20.4 mm
Other:
- net class cerocuatro added: clearance 0.2, trace_width 0.4, via_dia 0.8, via_drill 0.4
- net class cerotresmm added: clearance 0.2, trace_width 0.3, via_dia 0.8, via_drill 0.4
