File: ESP32_lamp/peripherals.sch (KiCad schematic (older format))
At the start: 31 parts, among them Q7 BSS214NW, Q8 BSS214NW, Q9 BSS214NW, U3 ADXL343, U4 AAAF5051-05, U5 AAAF5051-05, U6 AAAF5051-05

Commit message: update
Parts:
- added C12: 100nF, Capacitor_SMD:C_1206_3216Metric, symbol Device:C_Small
Connections:
- net 3V3: now also C12.1
- net GND: now also C12.2

Commit message: Release Candidate 0
Parts:
- added C13, C14, C15: 1uF, Capacitor_SMD:C_1206_3216Metric, symbol Device:C_Small
- renumbered U4 to LED1, U5 to LED2, U6 to LED3, Q7 to Q_B3, Q9 to Q_G3, Q8 to Q_R3
Connections:
- net 3V3_SW is gone; now on net 3V3: LED1.4, LED1.5, LED1.6, LED1.7 (Anodo), LED2.4, LED2.5, LED2.6, LED2.7 (Anodo), LED3.4, LED3.5, LED3.6, LED3.7 (Anodo)
- net 3V3: now also C13.1, C14.1, C15.1
- net GND: now also C13.2, C14.2, C15.2
Changed lines of the file:
@@
 	9800 2850 9800 4300
 Text GLabel 3200 1600 1    50   Input ~ 0
-3V3_SW
+3V3
 Text GLabel 6450 1150 1    50   Input ~ 0
-3V3_SW
+3V3
 Text GLabel 9200 1200 1    50   Input ~ 0
-3V3_SW
+3V3
 Wire Wire Line
 	2650 3300 2450 3300
@@
 AR Path="/5F23FCD8" Ref="Q?"  Part="1"
 AR Path="/5F10C517/5F23FCD8" Ref="Q?"  Part="1"
-AR Path="/5F289DCA/5F23FCD8" Ref="Q9"  Part="1"
-F 0 "Q9" H 9904 4546 50  0000 L CNN
+AR Path="/5F289DCA/5F23FCD8" Ref="Q_G3"  Part="1"
+F 0 "Q_G3" H 9904 4546 50  0000 L CNN
 F 1 "BSS214NW" H 9904 4455 50  0000 L CNN
 F 2 "Package_TO_SOT_SMD:SOT-323_SC-70" H 9900 4425 50  0001 L CIN
@@
 AR Path="/5F23FCDE" Ref="Q?"  Part="1"
 AR Path="/5F10C517/5F23FCDE" Ref="Q?"  Part="1"
-AR Path="/5F289DCA/5F23FCDE" Ref="Q8"  Part="1"
-F 0 "Q8" H 9704 3946 50  0000 L CNN
+AR Path="/5F289DCA/5F23FCDE" Ref="Q_R3"  Part="1"
+F 0 "Q_R3" H 9704 3946 50  0000 L CNN
 F 1 "BSS214NW" H 9704 3855 50  0000 L CNN
 F 2 "Package_TO_SOT_SMD:SOT-323_SC-70" H 9700 3825 50  0001 L CIN
@@
 AR Path="/5F23FCE4" Ref="Q?"  Part="1"
 AR Path="/5F10C517/5F23FCE4" Ref="Q?"  Part="1"
-AR Path="/5F289DCA/5F23FCE4" Ref="Q7"  Part="1"
-F 0 "Q7" H 9504 3396 50  0000 L CNN
+AR Path="/5F289DCA/5F23FCE4" Ref="Q_B3"  Part="1"
+F 0 "Q_B3" H 9504 3396 50  0000 L CNN
 F 1 "BSS214NW" H 9504 3305 50  0000 L CNN
 F 2 "Package_TO_SOT_SMD:SOT-323_SC-70" H 9500 3275 50  0001 L CIN
@@
 AR Path="/5F23FD90" Ref="U?"  Part="1"
 AR Path="/5F10C517/5F23FD90" Ref="U?"  Part="1"
-AR Path="/5F289DCA/5F23FD90" Ref="U6"  Part="1"
-F 0 "U6" V 9529 2228 50  0000 L CNN
+AR Path="/5F289DCA/5F23FD90" Ref="LED3"  Part="1"
+F 0 "LED3" V 9529 2228 50  0000 L CNN
 F 1 "AAAF5051-05" V 9620 2228 50  0000 L CNN
 F 2 "ESP32_lamp:kinbright-AAAF5051-05" H 9550 1400 50  0001 C CNN
@@
 AR Path="/5F23FD96" Ref="U?"  Part="1"
 AR Path="/5F10C517/5F23FD96" Ref="U?"  Part="1"
-AR Path="/5F289DCA/5F23FD96" Ref="U5"  Part="1"
-F 0 "U5" V 6779 2178 50  0000 L CNN
+AR Path="/5F289DCA/5F23FD96" Ref="LED2"  Part="1"
+F 0 "LED2" V 6779 2178 50  0000 L CNN
 F 1 "AAAF5051-05" V 6870 2178 50  0000 L CNN
 F 2 "ESP32_lamp:kinbright-AAAF5051-05" H 6800 1350 50  0001 C CNN
@@
 AR Path="/5F23FD9C" Ref="U?"  Part="1"
 AR Path="/5F10C517/5F23FD9C" Ref="U?"  Part="1"
-AR Path="/5F289DCA/5F23FD9C" Ref="U4"  Part="1"
-F 0 "U4" V 3529 2528 50  0000 L CNN
+AR Path="/5F289DCA/5F23FD9C" Ref="LED1"  Part="1"
+F 0 "LED1" V 3529 2528 50  0000 L CNN
 F 1 "AAAF5051-05" V 3620 2528 50  0000 L CNN
 F 2 "ESP32_lamp:kinbright-AAAF5051-05" H 3550 1700 50  0001 C CNN
@@
 	1    0    0    -1
 $EndComp
+$Comp
+L Device:C_Small C13
+U 1 1 5F397828
+P 2850 1950
+F 0 "C13" H 2942 1996 50  0000 L CNN
+F 1 "1uF" H 2942 1905 50  0000 L CNN
+F 2 "Capacitor_SMD:C_1206_3216Metric" H 2850 1950 50  0001 C CNN
+F 3 "~" H 2850 1950 50  0001 C CNN
+	1    2850 1950
+	1    0    0    -1
+$EndComp
+$Comp
+L power:GND #PWR?
+U 1 1 5F39E28C
+P 2850 2200
+AR Path="/5F39E28C" Ref="#PWR?"  Part="1"
+AR Path="/5F10C517/5F39E28C" Ref="#PWR?"  Part="1"
+AR Path="/5F289DCA/5F39E28C" Ref="#PWR0101"  Part="1"
+F 0 "#PWR0101" H 2850 1950 50  0001 C CNN
+F 1 "GND" H 2855 2027 50  0000 C CNN
+F 2 "" H 2850 2200 50  0001 C CNN
+F 3 "" H 2850 2200 50  0001 C CNN
+	1    2850 2200
+	1    0    0    -1
+$EndComp
+Wire Wire Line
+	2850 2200 2850 2050
+Wire Wire Line
+	2850 1850 2850 1700
+Wire Wire Line
+	2850 1700 3200 1700
+$Comp
+L Device:C_Small C14
+U 1 1 5F3A3A70
+P 6200 1800
+F 0 "C14" H 6292 1846 50  0000 L CNN
+F 1 "1uF" H 6292 1755 50  0000 L CNN
+F 2 "Capacitor_SMD:C_1206_3216Metric" H 6200 1800 50  0001 C CNN
+F 3 "~" H 6200 1800 50  0001 C CNN
+	1    6200 1800
+	1    0    0    -1
+$EndComp
+$Comp
+L power:GND #PWR?
+U 1 1 5F3A41AF
+P 6200 2000
+AR Path="/5F3A41AF" Ref="#PWR?"  Part="1"
+AR Path="/5F10C517/5F3A41AF" Ref="#PWR?"  Part="1"
+AR Path="/5F289DCA/5F3A41AF" Ref="#PWR0102"  Part="1"
+F 0 "#PWR0102" H 6200 1750 50  0001 C CNN
+F 1 "GND" H 6205 1827 50  0000 C CNN
+F 2 "" H 6200 2000 50  0001 C CNN
+F 3 "" H 6200 2000 50  0001 C CNN
+	1    6200 2000
+	1    0    0    -1
+$EndComp
+Wire Wire Line
+	6200 2000 6200 1900
+Wire Wire Line
+	6200 1700 6200 1350
+Wire Wire Line
+	6200 1350 6450 1350
+$Comp
+L Device:C_Small C15
+U 1 1 5F3A9E8B
+P 8950 1850
+F 0 "C15" H 9042 1896 50  0000 L CNN
+F 1 "1uF" H 9042 1805 50  0000 L CNN
+F 2 "Capacitor_SMD:C_1206_3216Metric" H 8950 1850 50  0001 C CNN
+F 3 "~" H 8950 1850 50  0001 C CNN
+	1    8950 1850
+	1    0    0    -1
+$EndComp
+$Comp
+L power:GND #PWR?
+U 1 1 5F3AA583
+P 8950 2050
+AR Path="/5F3AA583" Ref="#PWR?"  Part="1"
+AR Path="/5F10C517/5F3AA583" Ref="#PWR?"  Part="1"
+AR Path="/5F289DCA/5F3AA583" Ref="#PWR0103"  Part="1"
+F 0 "#PWR0103" H 8950 1800 50  0001 C CNN
+F 1 "GND" H 8955 1877 50  0000 C CNN
+F 2 "" H 8950 2050 50  0001 C CNN
+F 3 "" H 8950 2050 50  0001 C CNN
+	1    8950 2050
+	1    0    0    -1
+$EndComp
+Wire Wire Line
+	8950 1950 8950 2050
+Wire Wire Line
+	8950 1750 8950 1400
+Wire Wire Line
+	8950 1400 9200 1400
 $EndSCHEMATC

Commit message: WIP Release Candidate 1
Parts:
- R_R12, R_R22, R_R32: MPN (none) -> SG73P2BTTD6R8J; PD (none) -> 500mW
Changed lines of the file:
@@
 F 2 "Resistor_SMD:R_1206_3216Metric" V 9530 2700 50  0001 C CNN
 F 3 "~" H 9600 2700 50  0001 C CNN
+F 4 "SG73P2BTTD6R8J" V 9600 2700 50  0001 C CNN "MPN"
+F 5 "500mW" V 9600 2700 50  0001 C CNN "PD"
 	1    9600 2700
 	-1   0    0    1
@@
 F 2 "Resistor_SMD:R_1206_3216Metric" V 3530 2750 50  0001 C CNN
 F 3 "~" H 3600 2750 50  0001 C CNN
+F 4 "SG73P2BTTD6R8J" V 3600 2750 50  0001 C CNN "MPN"
+F 5 "500mW" V 3600 2750 50  0001 C CNN "PD"
 	1    3600 2750
 	-1   0    0    1
@@
 F 2 "Resistor_SMD:R_1206_3216Metric" V 6780 2550 50  0001 C CNN
 F 3 "~" H 6850 2550 50  0001 C CNN
+F 4 "SG73P2BTTD6R8J" V 6850 2550 50  0001 C CNN "MPN"
+F 5 "500mW" V 6850 2550 50  0001 C CNN "PD"
 	1    6850 2550
 	-1   0    0    1

Commit message: Release
Parts:
- LED1, LED2, LED3: footprint ESP32_lamp:kinbright-AAAF5051-05 -> ESP32_lamp:kinbright-AAAF5051-05_MOD
Changed lines of the file:
@@
 F 0 "LED3" V 9529 2228 50  0000 L CNN
 F 1 "AAAF5051-05" V 9620 2228 50  0000 L CNN
-F 2 "ESP32_lamp:kinbright-AAAF5051-05" H 9550 1400 50  0001 C CNN
+F 2 "ESP32_lamp:kinbright-AAAF5051-05_MOD" H 9550 1400 50  0001 C CNN
 F 3 "http://www.kingbrightusa.com/images/catalog/SPEC/AAAF5051-05.pdf" H 9600 1900 50  0001 C CNN
 	1    9600 1900
@@
 F 0 "LED2" V 6779 2178 50  0000 L CNN
 F 1 "AAAF5051-05" V 6870 2178 50  0000 L CNN
-F 2 "ESP32_lamp:kinbright-AAAF5051-05" H 6800 1350 50  0001 C CNN
+F 2 "ESP32_lamp:kinbright-AAAF5051-05_MOD" H 6800 1350 50  0001 C CNN
 F 3 "http://www.kingbrightusa.com/images/catalog/SPEC/AAAF5051-05.pdf" H 6850 1850 50  0001 C CNN
 	1    6850 1850
@@
 F 0 "LED1" V 3529 2528 50  0000 L CNN
 F 1 "AAAF5051-05" V 3620 2528 50  0000 L CNN
-F 2 "ESP32_lamp:kinbright-AAAF5051-05" H 3550 1700 50  0001 C CNN
+F 2 "ESP32_lamp:kinbright-AAAF5051-05_MOD" H 3550 1700 50  0001 C CNN
 F 3 "http://www.kingbrightusa.com/images/catalog/SPEC/AAAF5051-05.pdf" H 3600 2200 50  0001 C CNN
 	1    3600 2200
