File: kicad_files/ESP32_&_LEDS.sch (KiCad schematic (older format))
At the start: 14 parts, among them J2 Conn_02x05_Odd_Even, J4 Conn_01x03, SW1 SW_Push, U2 ESP32-WROOM-32D

Commit message: Update MPN attributes && BOM file
Parts:
- J2: MPN (none) -> M50-3610542R
- SW1: MPN (none) -> EVQ-PUJ02K
- U2: MPN (none) -> ESP32-WROOM-32D
Changed lines of the file:
@@
 F 2 "RF_Module:ESP32-WROOM-32" H 1900 2600 50  0001 C CNN
 F 3 "https://www.espressif.com/sites/default/files/documentation/esp32-wroom-32d_esp32-wroom-32u_datasheet_en.pdf" H 1600 4150 50  0001 C CNN
+F 4 "ESP32-WROOM-32D" H 1900 4100 50  0001 C CNN "MPN"
 	1    1900 4100
 	1    0    0    -1
@@
 F 2 "Connector_PinHeader_1.27mm:PinHeader_2x05_P1.27mm_Vertical_SMD" H 1600 6700 50  0001 C CNN
 F 3 "~" H 1600 6700 50  0001 C CNN
-F 4 "" H 1600 6700 50  0001 C CNN "MPN"
+F 4 "M50-3610542R" H 1600 6700 50  0001 C CNN "MPN"
 	1    1600 6700
 	1    0    0    -1
@@
 F 2 "Button_Switch_SMD:Panasonic_EVQPUJ_EVQPUA" H 5350 2600 50  0001 C CNN
 F 3 "~" H 5350 2600 50  0001 C CNN
+F 4 "EVQ-PUJ02K" H 5350 2400 50  0001 C CNN "MPN"
 	1    5350 2400
 	-1   0    0    -1
