File: kicad_files/ESP32_lamp.sch (KiCad schematic (older format))
At the start: 4 parts

Commit message: Update MPN attributes && BOM file
Parts:
- H1, H2, H3, H4: MPN (none) -> SJ-5003 (BLACK)
Changed lines of the file:
@@
 F 2 "MountingHole:MountingHole_3.2mm_M3_ISO7380" H 2450 7350 50  0001 C CNN
 F 3 "~" H 2450 7350 50  0001 C CNN
+F 4 "SJ-5003 (BLACK)" H 2450 7350 50  0001 C CNN "MPN"
 	1    2450 7350
 	1    0    0    -1
@@
 F 2 "MountingHole:MountingHole_3.2mm_M3_ISO7380" H 3000 7350 50  0001 C CNN
 F 3 "~" H 3000 7350 50  0001 C CNN
+F 4 "SJ-5003 (BLACK)" H 3000 7350 50  0001 C CNN "MPN"
 	1    3000 7350
 	1    0    0    -1
@@
 F 2 "MountingHole:MountingHole_3.2mm_M3_ISO7380" H 2450 7100 50  0001 C CNN
 F 3 "~" H 2450 7100 50  0001 C CNN
+F 4 "SJ-5003 (BLACK)" H 2450 7100 50  0001 C CNN "MPN"
 	1    2450 7100
 	1    0    0    -1
@@
 F 2 "MountingHole:MountingHole_3.2mm_M3_ISO7380" H 3000 7100 50  0001 C CNN
 F 3 "~" H 3000 7100 50  0001 C CNN
+F 4 "SJ-5003 (BLACK)" H 3000 7100 50  0001 C CNN "MPN"
 	1    3000 7100
 	1    0    0    -1
