File: kicad_files/Fuente_alimentacion.sch (KiCad schematic (older format))
At the start: 13 parts, among them J1 USB_B_Micro, U1 LMR33630BDDA

Commit message: Update MPN attributes && BOM file
Parts:
- J1: symbol Connector:USB_B_Micro -> ESP32_lamp-rescue:USB_B_Micro-Connector
- L1: MPN (none) -> TYS50402R2N-10
- U1: MPN (none) -> LMR33630BDDAR
Changed lines of the file:
@@
 F 2 "Inductor_SMD:L_Taiyo-Yuden_MD-5050" H 7000 3300 50  0001 C CNN
 F 3 "~" H 7000 3300 50  0001 C CNN
+F 4 "TYS50402R2N-10 " H 7000 3300 50  0001 C CNN "MPN"
 	1    7000 3300
 	0    -1   -1   0
@@
 	5200 4200 5200 4050
 $Comp
-L Connector:USB_B_Micro J1
+L ESP32_lamp-rescue:USB_B_Micro-Connector J1
 U 1 1 5F0D553A
 P 2550 3600
+AR Path="/5F0D553A" Ref="J1"  Part="1"
+AR Path="/5F0ACF9A/5F0D553A" Ref="J1"  Part="1"
 F 0 "J1" H 2607 4067 50  0000 C CNN
 F 1 "USB_B_Micro" H 2607 3976 50  0000 C CNN
@@
 F 2 "Package_SO:Texas_HSOP-8-1EP_3.9x4.9mm_P1.27mm_ThermalVias" H 5700 2700 50  0001 C CNN
 F 3 "http://www.ti.com/lit/ds/symlink/lmr33630.pdf" H 5700 3400 50  0001 C CNN
+F 4 "LMR33630BDDAR" H 5700 3500 50  0001 C CNN "MPN"
 	1    5700 3500
 	1    0    0    -1
