File: kicad_files/peripherals.sch (KiCad schematic (older format))
At the start: 35 parts, among them U3 ADXL343

Commit message: Update MPN attributes && BOM file
Parts:
- LED1, LED2, LED3: MPN (none) -> AAAF5051-05
- Q_B1, Q_B2, Q_B3, Q_G1, Q_G2, Q_G3, Q_R1, Q_R2, Q_R3: MPN (none) -> BSS214NWH6327XTSA1
- U3: MPN (none) -> ADXL343BCCZ
Changed lines of the file:
@@
 F 2 "Package_LGA:LGA-14_3x5mm_P0.8mm_LayoutBorder1x6y" H 2000 6550 50  0001 C CNN
 F 3 "https://www.analog.com/media/en/technical-documentation/data-sheets/ADXL343.pdf" H 2000 6550 50  0001 C CNN
+F 4 " ADXL343BCCZ" H 2000 6550 50  0001 C CNN "MPN"
 	1    2000 6550
 	1    0    0    -1
@@
 F 2 "Package_TO_SOT_SMD:SOT-323_SC-70" H 9900 4425 50  0001 L CIN
 F 3 "https://www.infineon.com/dgdl/Infineon-BSS214NW-DS-v02_02-en.pdf?fileId=db3a30431b3e89eb011b695aebc01bde" H 9700 4500 50  0001 L CNN
+F 4 "BSS214NWH6327XTSA1" H 9700 4500 50  0001 C CNN "MPN"
 	1    9700 4500
 	1    0    0    -1
@@
 F 2 "Package_TO_SOT_SMD:SOT-323_SC-70" H 9700 3825 50  0001 L CIN
 F 3 "https://www.infineon.com/dgdl/Infineon-BSS214NW-DS-v02_02-en.pdf?fileId=db3a30431b3e89eb011b695aebc01bde" H 9500 3900 50  0001 L CNN
+F 4 "BSS214NWH6327XTSA1" H 9500 3900 50  0001 C CNN "MPN"
 	1    9500 3900
 	1    0    0    -1
@@
 F 2 "Package_TO_SOT_SMD:SOT-323_SC-70" H 9500 3275 50  0001 L CIN
 F 3 "https://www.infineon.com/dgdl/Infineon-BSS214NW-DS-v02_02-en.pdf?fileId=db3a30431b3e89eb011b695aebc01bde" H 9300 3350 50  0001 L CNN
+F 4 "BSS214NWH6327XTSA1" H 9300 3350 50  0001 C CNN "MPN"
 	1    9300 3350
 	1    0    0    -1
@@
 F 2 "Package_TO_SOT_SMD:SOT-323_SC-70" H 7150 4425 50  0001 L CIN
 F 3 "https://www.infineon.com/dgdl/Infineon-BSS214NW-DS-v02_02-en.pdf?fileId=db3a30431b3e89eb011b695aebc01bde" H 6950 4500 50  0001 L CNN
+F 4 "BSS214NWH6327XTSA1" H 6950 4500 50  0001 C CNN "MPN"
 	1    6950 4500
 	1    0    0    -1
@@
 F 2 "Package_TO_SOT_SMD:SOT-323_SC-70" H 6950 3775 50  0001 L CIN
 F 3 "https://www.infineon.com/dgdl/Infineon-BSS214NW-DS-v02_02-en.pdf?fileId=db3a30431b3e89eb011b695aebc01bde" H 6750 3850 50  0001 L CNN
+F 4 "BSS214NWH6327XTSA1" H 6750 3850 50  0001 C CNN "MPN"
 	1    6750 3850
 	1    0    0    -1
@@
 F 2 "Package_TO_SOT_SMD:SOT-323_SC-70" H 6750 3125 50  0001 L CIN
 F 3 "https://www.infineon.com/dgdl/Infineon-BSS214NW-DS-v02_02-en.pdf?fileId=db3a30431b3e89eb011b695aebc01bde" H 6550 3200 50  0001 L CNN
+F 4 "BSS214NWH6327XTSA1" H 6550 3200 50  0001 C CNN "MPN"
 	1    6550 3200
 	1    0    0    -1
@@
 F 2 "Package_TO_SOT_SMD:SOT-323_SC-70" H 3900 4425 50  0001 L CIN
 F 3 "https://www.infineon.com/dgdl/Infineon-BSS214NW-DS-v02_02-en.pdf?fileId=db3a30431b3e89eb011b695aebc01bde" H 3700 4500 50  0001 L CNN
+F 4 "BSS214NWH6327XTSA1" H 3700 4500 50  0001 C CNN "MPN"
 	1    3700 4500
 	1    0    0    -1
@@
 F 2 "Package_TO_SOT_SMD:SOT-323_SC-70" H 3700 3825 50  0001 L CIN
 F 3 "https://www.infineon.com/dgdl/Infineon-BSS214NW-DS-v02_02-en.pdf?fileId=db3a30431b3e89eb011b695aebc01bde" H 3500 3900 50  0001 L CNN
+F 4 "BSS214NWH6327XTSA1" H 3500 3900 50  0001 C CNN "MPN"
 	1    3500 3900
 	1    0    0    -1
@@
 F 2 "Package_TO_SOT_SMD:SOT-323_SC-70" H 3500 3225 50  0001 L CIN
 F 3 "https://www.infineon.com/dgdl/Infineon-BSS214NW-DS-v02_02-en.pdf?fileId=db3a30431b3e89eb011b695aebc01bde" H 3300 3300 50  0001 L CNN
+F 4 "BSS214NWH6327XTSA1" H 3300 3300 50  0001 C CNN "MPN"
 	1    3300 3300
 	1    0    0    -1
@@
 F 2 "ESP32_lamp:kinbright-AAAF5051-05_MOD" H 9550 1400 50  0001 C CNN
 F 3 "http://www.kingbrightusa.com/images/catalog/SPEC/AAAF5051-05.pdf" H 9600 1900 50  0001 C CNN
+F 4 " AAAF5051-05" H 9600 1900 50  0001 C CNN "MPN"
 	1    9600 1900
 	0    1    1    0
@@
 F 2 "ESP32_lamp:kinbright-AAAF5051-05_MOD" H 6800 1350 50  0001 C CNN
 F 3 "http://www.kingbrightusa.com/images/catalog/SPEC/AAAF5051-05.pdf" H 6850 1850 50  0001 C CNN
+F 4 " AAAF5051-05" H 6850 1850 50  0001 C CNN "MPN"
 	1    6850 1850
 	0    1    1    0
@@
 F 2 "ESP32_lamp:kinbright-AAAF5051-05_MOD" H 3550 1700 50  0001 C CNN
 F 3 "http://www.kingbrightusa.com/images/catalog/SPEC/AAAF5051-05.pdf" H 3600 2200 50  0001 C CNN
+F 4 " AAAF5051-05" V 3600 2200 50  0001 C CNN "MPN"
 	1    3600 2200
 	0    1    1    0
