File: kicad_files/ESP32_lamp.kicad_pcb (KiCad board)
At the start: 2 copper layers, 70 x 70 mm, 66 parts, among them J1 USB_B_Micro, J2 Conn_02x05_Odd_Even, J4 Conn_01x03, SW1 SW_Push, U1 LMR33630BDDA, U2 ESP32-WROOM-32D, U3 ADXL343

Commit message: Release candidate
Parts:
- removed CB1: CircuitBreaker_1P_US, Jumper:SolderJumper-2_P1.3mm_Open_TrianglePad1.0x1.5mm
- added C17: 100nF, Capacitor_SMD:C_1206_3216Metric, B.Cu at (200.9, 128.0)
- added SW2: SW_Push, Button_Switch_SMD:Panasonic_EVQPUJ_EVQPUA, B.Cu at (187.9, 127.2)
- R6, R7: value 10k -> 100k
- moved J4 35.0 mm to (185.6, 92.6), turned to 180 degrees
- moved R6 29.0 mm to (201.2, 131.1)
Connections:
- J1 pad 2: Net-(J1-Pad2) -> unconnected-(J1-Pad2)
- J1 pad 3: Net-(J1-Pad3) -> unconnected-(J1-Pad3)
- J1 pad 4: Net-(J1-Pad4) -> unconnected-(J1-Pad4)
- J2 pad 10: Net-(J2-Pad10) -> unconnected-(J2-Pad10)
- R6 pad 1: Net-(CB1-Pad2) -> 3V3
- R6 pad 2: GND -> Net-(C17-Pad1)
- U1 pad 4: Net-(U1-Pad4) -> unconnected-(U1-Pad4)
- U2 pad 17: Net-(U2-Pad17) -> unconnected-(U2-Pad17)
- U2 pad 18: Net-(U2-Pad18) -> unconnected-(U2-Pad18)
- U2 pad 19: Net-(U2-Pad19) -> unconnected-(U2-Pad19)
- U2 pad 20: Net-(U2-Pad20) -> unconnected-(U2-Pad20)
- U2 pad 21: Net-(U2-Pad21) -> unconnected-(U2-Pad21)
- U2 pad 22: Net-(U2-Pad22) -> unconnected-(U2-Pad22)
- U2 pad 24: Net-(U2-Pad24) -> unconnected-(U2-Pad24)
- U2 pad 29: Net-(U2-Pad29) -> unconnected-(U2-Pad29)
- U2 pad 32: Net-(U2-Pad32) -> unconnected-(U2-Pad32)
- U2 pad 4: Net-(U2-Pad4) -> unconnected-(U2-Pad4)
- U2 pad 5: Net-(U2-Pad5) -> unconnected-(U2-Pad5)
- U2 pad 6: Net-(U2-Pad6) -> unconnected-(U2-Pad6)
- U2 pad 7: Net-(U2-Pad7) -> unconnected-(U2-Pad7)
- U3 pad 10: Net-(U3-Pad10) -> unconnected-(U3-Pad10)
Routing:
- net 3V3: track 113.8 -> 271.2 mm
- net Net-(J4-Pad2): track 26.3 -> 3.68 mm
- net Net-(J4-Pad1): track 20.4 -> 4.25 mm
- net GND: track 141.8 -> 129.8 mm, vias 42 -> 41
- net Net-(C16-Pad1): track 33.0 -> 30.2 mm
- net INT2: track 13.7 -> 16.3 mm, vias 2 -> 0
- net INT1: track 14.4 -> 16.5 mm, vias 2 -> 0
- net Net-(CB1-Pad2): track 1.88 -> 0.00 mm
- net Net-(C17-Pad1): vias 0 -> 1
- added copper zone on F.Cu, net GND
- removed copper zone on F.Cu, net 3V3
Other:
- net class Default removed
- net class cerocuatro removed
- net class cerotresmm removed
- net class mediomm removed
